Commit message: Update urdf

File: diablo_A1/urdfs/diablo_robot/diablo_original/urdf/diablo_mesh.urdf (robot description, URDF)
Before this commit: robot diablo_mesh, 15 links, 14 joints
Links:
- link base_link: geometry collision mesh filename=../meshes/base_link.STL; visual mesh filename=../meshes/base_link.STL
- link left_leg1: geometry collision mesh filename=../meshes/left_leg1.STL; visual mesh filename=../meshes/left_leg1.STL
- link left_leg2: geometry collision mesh filename=../meshes/left_leg2.STL; visual mesh filename=../meshes/left_leg2.STL
- link left_leg3: geometry collision mesh filename=../meshes/left_leg3.STL; visual mesh filename=../meshes/left_leg3.STL
- link left_motor: geometry collision mesh filename=../meshes/left_motor.STL; visual mesh filename=../meshes/left_motor.STL
- link left_wheel: geometry collision mesh filename=../meshes/left_wheel.STL; visual mesh filename=../meshes/left_wheel.STL
- link little_wheel_left1: geometry collision mesh filename=../meshes/little_wheel_left1.STL; visual mesh filename=../meshes/little_wheel_left1.STL
- link little_wheel_left2: geometry collision mesh filename=../meshes/little_wheel_left2.STL; visual mesh filename=../meshes/little_wheel_left2.STL
- link little_wheel_right1: geometry collision mesh filename=../meshes/little_wheel_right1.STL; visual mesh filename=../meshes/little_wheel_right1.STL
- link little_wheel_right2: geometry collision mesh filename=../meshes/little_wheel_right2.STL; visual mesh filename=../meshes/little_wheel_right2.STL
- link right_leg1: geometry collision mesh filename=../meshes/right_leg1.STL; visual mesh filename=../meshes/right_leg1.STL
- link right_leg2: geometry collision mesh filename=../meshes/right_leg2.STL; visual mesh filename=../meshes/right_leg2.STL
- link right_leg3: geometry collision mesh filename=../meshes/right_leg3.STL; visual mesh filename=../meshes/right_leg3.STL
- link right_motor: geometry collision mesh filename=../meshes/right_motor.STL; visual mesh filename=../meshes/right_motor.STL
- link right_wheel: geometry collision mesh filename=../meshes/right_wheel.STL; visual mesh filename=../meshes/right_wheel.STL
